Commit message: Enabled movement in navigation for a1

File: src/enamour/a1_description/urdf/a1.urdf (robot description, URDF)
Before this commit: robot a1_description, 25 links, 24 joints
Links:
- removed link camera_face
- removed link camera_optical_face
- link trunk: mass 6.0 -> 4.713
Joints:
- removed joint camera_joint_face
- removed joint camera_optical_joint_face
- joint FL_calf_joint: limit lower=-2.69653369433 upper=-0.916297857297 effort=33.5 velocity=21 -> lower=-2.69653369433 upper=-0.916297857297 effort=55 velocity=28.6
- joint FL_hip_joint: limit lower=-0.802851455917 upper=0.802851455917 effort=33.5 velocity=21 -> lower=-0.802851455917 upper=0.802851455917 effort=20 velocity=52.4; origin xyz=0.1805 0.047 0 rpy=0 0 0 -> xyz=0.183 0.047 0 rpy=0 0 0
- joint FL_thigh_joint: limit lower=-1.0471975512 upper=4.18879020479 effort=33.5 velocity=21 -> lower=-1.0471975512 upper=4.18879020479 effort=55 velocity=28.6; origin xyz=0 0.0838 0 rpy=0 0 0 -> xyz=0 0.08505 0 rpy=0 0 0
- joint FR_calf_joint: limit lower=-2.69653369433 upper=-0.916297857297 effort=33.5 velocity=21 -> lower=-2.69653369433 upper=-0.916297857297 effort=55 velocity=28.6
- joint FR_hip_joint: limit lower=-0.802851455917 upper=0.802851455917 effort=33.5 velocity=21 -> lower=-0.802851455917 upper=0.802851455917 effort=20 velocity=52.4; origin xyz=0.1805 -0.047 0 rpy=0 0 0 -> xyz=0.183 -0.047 0 rpy=0 0 0
- joint FR_thigh_joint: limit lower=-1.0471975512 upper=4.18879020479 effort=33.5 velocity=21 -> lower=-1.0471975512 upper=4.18879020479 effort=55 velocity=28.6; origin xyz=0 -0.0838 0 rpy=0 0 0 -> xyz=0 -0.08505 0 rpy=0 0 0
- joint RL_calf_joint: limit lower=-2.69653369433 upper=-0.916297857297 effort=33.5 velocity=21 -> lower=-2.69653369433 upper=-0.916297857297 effort=55 velocity=28.6
- joint RL_hip_joint: limit lower=-0.802851455917 upper=0.802851455917 effort=33.5 velocity=21 -> lower=-0.802851455917 upper=0.802851455917 effort=20 velocity=52.4; origin xyz=-0.1805 0.047 0 rpy=0 0 0 -> xyz=-0.183 0.047 0 rpy=0 0 0
- joint RL_thigh_joint: limit lower=-1.0471975512 upper=4.18879020479 effort=33.5 velocity=21 -> lower=-1.0471975512 upper=4.18879020479 effort=55 velocity=28.6; origin xyz=0 0.0838 0 rpy=0 0 0 -> xyz=0 0.08505 0 rpy=0 0 0
- joint RR_calf_joint: limit lower=-2.69653369433 upper=-0.916297857297 effort=33.5 velocity=21 -> lower=-2.69653369433 upper=-0.916297857297 effort=55 velocity=28.6
- joint RR_hip_joint: limit lower=-0.802851455917 upper=0.802851455917 effort=33.5 velocity=21 -> lower=-0.802851455917 upper=0.802851455917 effort=20 velocity=52.4; origin xyz=-0.1805 -0.047 0 rpy=0 0 0 -> xyz=-0.183 -0.047 0 rpy=0 0 0
- joint RR_thigh_joint: limit lower=-1.0471975512 upper=4.18879020479 effort=33.5 velocity=21 -> lower=-1.0471975512 upper=4.18879020479 effort=55 velocity=28.6; origin xyz=0 -0.0838 0 rpy=0 0 0 -> xyz=0 -0.08505 0 rpy=0 0 0

File: src/enamour/a1_description/xacro/robot.xacro (robot description, xacro)
@@ -5,7 +5,5 @@
     <xacro:include filename="$(find a1_description)/xacro/leg.xacro"/>
     <xacro:include filename="$(find a1_description)/xacro/stairs.xacro"/>
-    <xacro:include filename="$(find a1_description)/xacro/depthCamera.xacro"/>
-    <xacro:include filename="$(find a1_description)/xacro/_d435i.urdf.xacro"/>
-    <xacro:include filename="$(find a1_description)/xacro/gazebo.xacro"/>
+    <!-- <xacro:include filename="$(find a1_gazebo)/launch/gazebo.xacro"/> -->
     <!-- <xacro:include filename="$(find a1_gazebo)/launch/stairs.urdf.xacro"/> -->
     <!-- <xacro:stairs stairs="15" xpos="0" ypos="0" zpos="0" /> -->
@@ -123,7 +121,4 @@
         <origin rpy="0 0 0" xyz="${-leg_offset_x} ${leg_offset_y} 0"/>
     </xacro:leg>
-     <xacro:depthCamera camID="1" name="face">
-        <origin rpy="${PI} 0 0" xyz="0.2785 0.0125 0.0167"/>
-    </xacro:depthCamera>
     <!-- <xacro:stairs stairs="15" xpos="0" ypos="2.0" zpos="0" /> -->
 </robot>
